File: LoRa-Module/LoRa-Module.kicad_pcb (KiCad board)
At the start: 2 copper layers, 34.9 x 34.9 mm, 13 parts, among them J1 Conn_01x09, J2 Conn_01x05, J3 Conn_Coaxial, J4 Conn_01x01, J5 Conn_01x01, J6 Conn_01x01, J7 Conn_01x01, U1 AZ1117-3.3, U2 74HC4050D, U3 RFM98

Commit message: fixed gerber error
Routing:
- net GND: track 27.1 -> 92.1 mm, vias 6 -> 12
- net (no net): track 3.18 -> 0.00 mm, vias 8 -> 0
- net /DIO3: track 30.1 -> 30.6 mm
